File: hardware/ExpressionController.kicad_pcb (KiCad board)
At the start: 2 copper layers, 86.6 x 72.6 mm, 130 parts, among them J1 DC, J2 Exp1, J3 Exp2, J4 Exp3, J5 Exp4, Q1 DMP3099L-7, U1 ADP7142AUJZ-3.3, U10 74HC595, U12 74HC595, U14 74AHCT1G125, U15 TMUX1511PWR, U16 TMUX1511PWR, U17 TMUX1511PWR, U18 TMUX1511PWR, U19 TMUX1511PWR, U2 ADP7142AUJZ-5.0, U20 TMUX1511PWR, U21 TMUX1511PWR, U22 TMUX1511PWR, U3 ADP7142AUJZ-2.5, U4 AD7718, U5 AD7718, U6 74HC595, U8 74HC595, Y1 MS1V-T1K-32.768kHz-12.5pF-20P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, Y2 MS1V-T1K-32.768kHz-12.5pF-20P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

Commit message: new PCB updates
Parts:
- C10: footprint Capacitor_SMD:C_1210_3225Metric -> Capacitor_SMD:C_0805_2012Metric
- C53, C54, C57, C58, C59, C60, R51, R52, R53, R54, R55, R56, R57, U16, U17, U18, U20, U21, U22: moved to B.Cu
- moved R55 157.0 mm to (143.5, 172.5)
- moved C57 151.1 mm to (133.3, 171.4), turned to 90 degrees
- moved R51 149.2 mm to (149.6, 162.1), turned to -90 degrees
- moved C58 145.6 mm to (154.7, 173.0), turned to 90 degrees
- moved U16 143.5 mm to (149.6, 166.6)
- moved U20 143.2 mm to (149.6, 172.2)
- moved U17 119.1 mm to (170.9, 166.6)
- moved U21 118.9 mm to (170.9, 172.2)
- moved C49 105.7 mm to (123.7, 190.0), turned to -90 degrees
- moved U8 91.4 mm to (149.6, 182.1), turned to -90 degrees
- moved U10 84.4 mm to (170.9, 182.1), turned to -90 degrees
- moved U12 83.9 mm to (192.3, 182.1), turned to -90 degrees
- moved U18 83.6 mm to (192.3, 166.6)
- moved U22 83.3 mm to (192.3, 172.2)
- moved C54 79.3 mm to (154.7, 167.4)
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Connections:
- U15 pad 11: /AnalogFrontend/AnalogQuadChannel1/JACK4 -> /AnalogFrontend/AnalogQuadChannel1/JACK2
- U15 pad 3: /AnalogFrontend/AnalogQuadChannel1/JACK1 -> /AnalogFrontend/AnalogQuadChannel1/JACK3
- U15 pad 6: /AnalogFrontend/AnalogQuadChannel1/JACK2 -> /AnalogFrontend/AnalogQuadChannel1/JACK4
- U15 pad 8: /AnalogFrontend/AnalogQuadChannel1/JACK3 -> /AnalogFrontend/AnalogQuadChannel1/JACK1
- U16 pad 11: /AnalogFrontend/AnalogQuadChannel2/JACK4 -> /AnalogFrontend/AnalogQuadChannel2/JACK2
- U16 pad 3: /AnalogFrontend/AnalogQuadChannel2/JACK1 -> /AnalogFrontend/AnalogQuadChannel2/JACK3
- U16 pad 6: /AnalogFrontend/AnalogQuadChannel2/JACK2 -> /AnalogFrontend/AnalogQuadChannel2/JACK4
- U16 pad 8: /AnalogFrontend/AnalogQuadChannel2/JACK3 -> /AnalogFrontend/AnalogQuadChannel2/JACK1
- U17 pad 1: Net-(U10-QC) -> Net-(U10-QB)
- U17 pad 10: Net-(U10-QA) -> Net-(U10-QH)
- U17 pad 11: /AnalogFrontend/AnalogQuadChannel3/JACK4 -> /AnalogFrontend/AnalogQuadChannel3/JACK2
- U17 pad 13: Net-(U10-QB) -> Net-(U10-QG)
- U17 pad 3: /AnalogFrontend/AnalogQuadChannel3/JACK1 -> /AnalogFrontend/AnalogQuadChannel3/JACK3
- U17 pad 4: Net-(U10-QD) -> Net-(U10-QA)
- U17 pad 6: /AnalogFrontend/AnalogQuadChannel3/JACK2 -> /AnalogFrontend/AnalogQuadChannel3/JACK4
- U17 pad 8: /AnalogFrontend/AnalogQuadChannel3/JACK3 -> /AnalogFrontend/AnalogQuadChannel3/JACK1
- U18 pad 1: Net-(U12-QC) -> Net-(U12-QB)
- U18 pad 10: Net-(U12-QA) -> Net-(U12-QH)
- U18 pad 11: /AnalogFrontend/AnalogQuadChannel4/JACK4 -> /AnalogFrontend/AnalogQuadChannel4/JACK2
- U18 pad 13: Net-(U12-QB) -> Net-(U12-QG)
- U18 pad 3: /AnalogFrontend/AnalogQuadChannel4/JACK1 -> /AnalogFrontend/AnalogQuadChannel4/JACK3
- U18 pad 4: Net-(U12-QD) -> Net-(U12-QA)
- U18 pad 6: /AnalogFrontend/AnalogQuadChannel4/JACK2 -> /AnalogFrontend/AnalogQuadChannel4/JACK4
- U18 pad 8: /AnalogFrontend/AnalogQuadChannel4/JACK3 -> /AnalogFrontend/AnalogQuadChannel4/JACK1
- U19 pad 11: /AnalogFrontend/AnalogQuadChannel1/JACK4 -> /AnalogFrontend/AnalogQuadChannel1/JACK2
- U19 pad 3: /AnalogFrontend/AnalogQuadChannel1/JACK1 -> /AnalogFrontend/AnalogQuadChannel1/JACK3
- U19 pad 6: /AnalogFrontend/AnalogQuadChannel1/JACK2 -> /AnalogFrontend/AnalogQuadChannel1/JACK4
- U19 pad 8: /AnalogFrontend/AnalogQuadChannel1/JACK3 -> /AnalogFrontend/AnalogQuadChannel1/JACK1
- U20 pad 11: /AnalogFrontend/AnalogQuadChannel2/JACK4 -> /AnalogFrontend/AnalogQuadChannel2/JACK2
- U20 pad 3: /AnalogFrontend/AnalogQuadChannel2/JACK1 -> /AnalogFrontend/AnalogQuadChannel2/JACK3
- U20 pad 6: /AnalogFrontend/AnalogQuadChannel2/JACK2 -> /AnalogFrontend/AnalogQuadChannel2/JACK4
- U20 pad 8: /AnalogFrontend/AnalogQuadChannel2/JACK3 -> /AnalogFrontend/AnalogQuadChannel2/JACK1
- U21 pad 1: Net-(U10-QE) -> Net-(U10-QD)
- U21 pad 10: Net-(U10-QG) -> Net-(U10-QF)
- U21 pad 11: /AnalogFrontend/AnalogQuadChannel3/JACK4 -> /AnalogFrontend/AnalogQuadChannel3/JACK2
- U21 pad 13: Net-(U10-QH) -> Net-(U10-QE)
- U21 pad 3: /AnalogFrontend/AnalogQuadChannel3/JACK1 -> /AnalogFrontend/AnalogQuadChannel3/JACK3
- U21 pad 4: Net-(U10-QF) -> Net-(U10-QC)
- U21 pad 6: /AnalogFrontend/AnalogQuadChannel3/JACK2 -> /AnalogFrontend/AnalogQuadChannel3/JACK4
- U21 pad 8: /AnalogFrontend/AnalogQuadChannel3/JACK3 -> /AnalogFrontend/AnalogQuadChannel3/JACK1
- U22 pad 1: Net-(U12-QE) -> Net-(U12-QD)
- U22 pad 10: Net-(U12-QG) -> Net-(U12-QF)
- U22 pad 11: /AnalogFrontend/AnalogQuadChannel4/JACK4 -> /AnalogFrontend/AnalogQuadChannel4/JACK2
- U22 pad 13: Net-(U12-QH) -> Net-(U12-QE)
- U22 pad 3: /AnalogFrontend/AnalogQuadChannel4/JACK1 -> /AnalogFrontend/AnalogQuadChannel4/JACK3
- U22 pad 4: Net-(U12-QF) -> Net-(U12-QC)
- U22 pad 6: /AnalogFrontend/AnalogQuadChannel4/JACK2 -> /AnalogFrontend/AnalogQuadChannel4/JACK4
- U22 pad 8: /AnalogFrontend/AnalogQuadChannel4/JACK3 -> /AnalogFrontend/AnalogQuadChannel4/JACK1
- U4 pad 1: /AnalogFrontend/AnalogQuadChannel2/ADC3 -> /AnalogFrontend/AnalogQuadChannel1/ADC3
- U4 pad 10: /AnalogFrontend/AnalogQuadChannel1/ADC4 -> /AnalogFrontend/AnalogQuadChannel2/ADC3
- U4 pad 11: /AnalogFrontend/AnalogQuadChannel2/ADC1 -> /AnalogFrontend/AnalogQuadChannel2/ADC4
- U4 pad 2: /AnalogFrontend/AnalogQuadChannel2/ADC4 -> /AnalogFrontend/AnalogQuadChannel1/ADC1
- U4 pad 7: /AnalogFrontend/AnalogQuadChannel1/ADC1 -> /AnalogFrontend/AnalogQuadChannel1/ADC2
- U4 pad 8: /AnalogFrontend/AnalogQuadChannel1/ADC2 -> /AnalogFrontend/AnalogQuadChannel1/ADC4
- U4 pad 9: /AnalogFrontend/AnalogQuadChannel1/ADC3 -> /AnalogFrontend/AnalogQuadChannel2/ADC1
- U5 pad 1: /AnalogFrontend/AnalogQuadChannel4/ADC3 -> /AnalogFrontend/AnalogQuadChannel3/ADC3
- U5 pad 10: /AnalogFrontend/AnalogQuadChannel3/ADC4 -> /AnalogFrontend/AnalogQuadChannel4/ADC3
- U5 pad 11: /AnalogFrontend/AnalogQuadChannel4/ADC1 -> /AnalogFrontend/AnalogQuadChannel4/ADC4
- U5 pad 2: /AnalogFrontend/AnalogQuadChannel4/ADC4 -> /AnalogFrontend/AnalogQuadChannel3/ADC1
- U5 pad 7: /AnalogFrontend/AnalogQuadChannel3/ADC1 -> /AnalogFrontend/AnalogQuadChannel3/ADC2
- U5 pad 8: /AnalogFrontend/AnalogQuadChannel3/ADC2 -> /AnalogFrontend/AnalogQuadChannel3/ADC4
- U5 pad 9: /AnalogFrontend/AnalogQuadChannel3/ADC3 -> /AnalogFrontend/AnalogQuadChannel4/ADC1
- U6 pad 1: Net-(U15-SEL4) -> Net-(U15-SEL1)
- U6 pad 15: Net-(U15-SEL3) -> Net-(U15-SEL2)
- U6 pad 2: Net-(U15-SEL1) -> Net-(U19-SEL2)
- U6 pad 3: Net-(U15-SEL2) -> Net-(U19-SEL1)
- U6 pad 4: Net-(U19-SEL1) -> Net-(U19-SEL4)
- U6 pad 5: Net-(U19-SEL2) -> Net-(U19-SEL3)
- U6 pad 6: Net-(U19-SEL3) -> Net-(U15-SEL4)
- U6 pad 7: Net-(U19-SEL4) -> Net-(U15-SEL3)
- U8 pad 1: Net-(U16-SEL4) -> Net-(U16-SEL1)
- U8 pad 15: Net-(U16-SEL3) -> Net-(U16-SEL2)
- U8 pad 2: Net-(U16-SEL1) -> Net-(U20-SEL2)
- U8 pad 3: Net-(U16-SEL2) -> Net-(U20-SEL1)
- U8 pad 4: Net-(U20-SEL1) -> Net-(U20-SEL4)
- U8 pad 5: Net-(U20-SEL2) -> Net-(U20-SEL3)
- U8 pad 6: Net-(U20-SEL3) -> Net-(U16-SEL4)
- U8 pad 7: Net-(U20-SEL4) -> Net-(U16-SEL3)
Routing:
- net +2.5V: track 0.00 -> 80.4 mm, vias 0 -> 4
- net /AnalogFrontend/AnalogQuadChannel2/JACK3: track 0.00 -> 30.6 mm, vias 0 -> 2
- net /AnalogFrontend/AnalogQuadChannel1/ADC4: track 2.20 -> 32.5 mm
- net /AnalogFrontend/AnalogQuadChannel2/ADC1: track 0.00 -> 29.6 mm
- net +3.3VA: track 0.00 -> 26.1 mm, vias 0 -> 2
- net Net-(U16-SEL2): track 0.00 -> 25.8 mm
- net /AnalogFrontend/AnalogQuadChannel2/JACK2: track 0.00 -> 23.9 mm, vias 0 -> 2
- net Net-(U16-SEL3): track 0.00 -> 20.8 mm
- net Net-(U16-SEL4): track 0.00 -> 20.7 mm
- net /AnalogFrontend/AnalogQuadChannel2/JACK1: track 0.00 -> 18.9 mm, vias 0 -> 2
- net Net-(U20-S1): track 0.00 -> 18.1 mm, vias 0 -> 1
- net Net-(U15-SEL2): track 8.31 -> 25.8 mm
- net /AnalogFrontend/AnalogQuadChannel1/ADC2: track 2.20 -> 19.4 mm
- net /AnalogFrontend/AnalogQuadChannel2/JACK4: track 0.00 -> 16.8 mm, vias 0 -> 2
- net /AnalogFrontend/AnalogQuadChannel2/ADC3: track 0.00 -> 16.7 mm
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- added copper zone on B.Cu, net GND
- added copper zone on F.Cu, net GND
