File: hardware/AnalogQuadChannel.kicad_sch (KiCad schematic)
At the start: 16 parts, among them U15 TMUX1511PWR, U19 TMUX1511PWR, U6 74HC595DR

Commit message: added all footprints and parts
Parts:
- U6: footprint Package_SO:SOIC-16W_7.5x10.3mm_P1.27mm -> Package_SO:SOIC-16_3.9x9.9mm_P1.27mm; Notes TODO: swap footprint -> (none)
Changed lines of the file:
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@@
 			)
 		)
-		(property "Footprint" "Package_SO:SOIC-16W_7.5x10.3mm_P1.27mm"
+		(property "Footprint" "Package_SO:SOIC-16_3.9x9.9mm_P1.27mm"
 			(at 59.69 101.6 0)
 			(hide yes)
@@
 			)
 		)
-		(property "Notes" "TODO: swap footprint"
+		(property "Notes" ""
 			(at 59.69 101.6 0)
 			(hide yes)

Commit message: more routing
Parts:
- R50, R54: Mouser No (none) -> ERA-6AEB102V; Part Source Uni/Mouser -> Mouser
Changed lines of the file:
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@@
 			)
 		)
-		(property "Mouser No" ""
+		(property "Mouser No" "ERA-6AEB102V"
 			(at 109.22 163.83 0)
 			(hide yes)
@@
 			)
 		)
-		(property "Part Source" "Uni/Mouser"
+		(property "Part Source" "Mouser"
 			(at 109.22 163.83 0)
 			(hide yes)
@@
 			)
 		)
-		(property "Mouser No" ""
+		(property "Mouser No" "ERA-6AEB102V"
 			(at 106.68 105.41 0)
 			(hide yes)
@@
 			)
 		)
-		(property "Part Source" "Uni/Mouser"
-			(at 106.68 105.41 0)
-			(hide yes)
+		(property "Part Source" "Mouser"
+			(at 106.68 105.41 0)
+			(hide yes)

Commit message: generated final assembly files
Changed lines of the file:
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@@
 		(in_pos_files yes)
 		(dnp no)
+		(fields_autoplaced yes)
 		(property "Reference" "#PWR036"
 			(at 50.8 99.06 0)
@@
 					(size 1.27 1.27)
 				)
-				(justify right)
+				(justify left)
 			)
 		)

Commit message: added signed declaration and updated schematic names
Other:
- company: (none) -> Amon Benson, TU Berlin
- title: (none) -> Jack Channel
Changed lines of the file:
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@@
 	(generator_version "10.0")
 	(paper "A4")
+	(title_block
+		(title "Jack Channel")
+		(date "2026-09-27")
+		(rev "1.0")
+		(company "Amon Benson, TU Berlin")
+	)
 	(text "Analog filter secion: around 1.6 kHz Cutoff\nUse low-tolerance components"
 		(exclude_from_sim no)

Commit message: some minor changes
Other:
- note added: "Analog filter section: around 1.6 kHz Cutoff Use low-tolerance components"
- note removed: "Analog filter secion: around 1.6 kHz Cutoff Use low-tolerance components"
Changed lines of the file:
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@@
 		(company "Amon Benson, TU Berlin")
 	)
-	(text "Analog filter secion: around 1.6 kHz Cutoff\nUse low-tolerance components"
+	(text "Analog filter section: around 1.6 kHz Cutoff\nUse low-tolerance components"
 		(exclude_from_sim no)
 		(at 193.04 24.13 0)
